File: hardware/bms.kicad_pcb (KiCad board)
At the start: 2 copper layers, 100 x 67 mm, 52 parts, among them IC1 BQ76920, IC2 LD1117S33TR, IC3 24LC256, P1 BAT, P2 LOAD, P3 CONN_01X05, P4 CONN_02X06, P5 CONN_02X09, P6 CONN_02X09, Q1 NMOS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

Commit message: Fix regulator grounding issue on PCB
Parts:
- IC2: value LD1117S33TR -> LD1117S33TR_SOT223
Connections:
- C14 pad 2: Net-(C14-Pad2) -> GND
- C15 pad 2: Net-(C14-Pad2) -> GND
- IC1 pad 11: Net-(IC1-Pad11) -> (no net)
- IC2 pad 1: Net-(C14-Pad2) -> GND
- P5 pad 10: Net-(P5-Pad10) -> (no net)
- P5 pad 13: Net-(P5-Pad13) -> (no net)
- P5 pad 16: Net-(P5-Pad16) -> (no net)
- P5 pad 17: Net-(P5-Pad17) -> (no net)
- P5 pad 18: Net-(P5-Pad18) -> (no net)
- P5 pad 4: Net-(P5-Pad4) -> (no net)
- P5 pad 5: Net-(P5-Pad5) -> (no net)
- P5 pad 6: Net-(P5-Pad6) -> (no net)
- P5 pad 7: Net-(P5-Pad7) -> (no net)
- P5 pad 8: Net-(P5-Pad8) -> (no net)
- P5 pad 9: Net-(P5-Pad9) -> (no net)
- P6 pad 10: Net-(P6-Pad10) -> (no net)
- P6 pad 12: Net-(P6-Pad12) -> (no net)
- P6 pad 14: Net-(P6-Pad14) -> (no net)
- P6 pad 15: Net-(P6-Pad15) -> (no net)
- P6 pad 16: Net-(P6-Pad16) -> (no net)
- P6 pad 17: Net-(P6-Pad17) -> (no net)
- P6 pad 18: Net-(P6-Pad18) -> (no net)
- P6 pad 2: Net-(P6-Pad2) -> (no net)
- P6 pad 3: Net-(P6-Pad3) -> (no net)
- P6 pad 4: Net-(P6-Pad4) -> (no net)
- P6 pad 7: Net-(P6-Pad7) -> (no net)
- P6 pad 8: Net-(P6-Pad8) -> (no net)
- P6 pad 9: Net-(P6-Pad9) -> (no net)
Routing:
- net Net-(C14-Pad2): track 7.78 -> 0.00 mm
- net GND: track 67.5 -> 75.3 mm
